File: KiCad/SEIENTS_EDD.kicad_sch (KiCad schematic)
At the start: 0 parts

Commit message: Primer Esquematic
Other:
- added sheet ALIMENTACIO (ALIMENTACIO.kicad_sch)
- added sheet MICROCONTROLADOR (MICROCONTROLADOR.kicad_sch)
- note added: "ALIMENTACIO"
- note added: "MICROCONTROLADOR"
Changed lines of the file:
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@@
 	(generator_version "9.0")
 	(paper "A4")
+	(text "ALIMENTACIO"
+		(exclude_from_sim no)
+		(at 62.738 62.484 0)
+		(effects
+			(font
+				(size 5.08 5.08)
+			)
+		)
+	)
+	(text "MICROCONTROLADOR\n"
+		(exclude_from_sim no)
+		(at 131.064 63.246 0)
+		(effects
+			(font
+				(size 3.81 3.81)
+			)
+		)
+	)
+	(sheet
+		(at 99.06 27.94)
+		(size 63.5 71.12)
+		(exclude_from_sim no)
+		(in_bom yes)
+		(on_board yes)
+		(dnp no)
+		(fields_autoplaced yes)
+		(stroke
+			(width 0.1524)
+			(type solid)
+		)
+		(fill
+			(color 0 0 0 0.0000)
+		)
+		(property "Sheetname" "MICROCONTROLADOR"
+			(at 99.06 27.2284 0)
+			(effects
+				(font
+					(size 1.27 1.27)
+				)
+				(justify left bottom)
+			)
+		)
+		(property "Sheetfile" "MICROCONTROLADOR.kicad_sch"
+			(at 99.06 99.6446 0)
+			(effects
+				(font
+					(size 1.27 1.27)
+				)
+				(justify left top)
+			)
+		)
+		(instances
+			(project "SEIENTS_EDD"
+				(path "/b6401b4f-5426-49b8-bb2e-8ecdb19989ef"
+					(page "3")
+				)
+			)
+		)
+	)
+	(sheet
+		(at 31.75 27.94)
+		(size 62.23 71.12)
+		(exclude_from_sim no)
+		(in_bom yes)
+		(on_board yes)
+		(dnp no)
+		(fields_autoplaced yes)
+		(stroke
+			(width 0.1524)
+			(type solid)
+		)
+		(fill
+			(color 0 0 0 0.0000)
+		)
+		(property "Sheetname" "ALIMENTACIO"
+			(at 31.75 27.2284 0)
+			(effects
+				(font
+					(size 1.27 1.27)
+				)
+				(justify left bottom)
+			)
+		)
+		(property "Sheetfile" "ALIMENTACIO.kicad_sch"
+			(at 31.75 99.6446 0)
+			(effects
+				(font
+					(size 1.27 1.27)
+				)
+				(justify left top)
+			)
+		)
+		(instances
+			(project "SEIENTS_EDD"
+				(path "/b6401b4f-5426-49b8-bb2e-8ecdb19989ef"
+					(page "2")
+				)
+			)
+		)
+	)
 	(sheet_instances
 		(path "/"
