File: KiCad/DRIVERS(MOTORS).kicad_sch (KiCad schematic)
At the start: 17 parts, among them M1 Motor_DC, M2 Motor_DC, M3 Motor_DC, U11 ATtiny1616-M, U12 DRV8871DDA, U6 TB6612FNG

Commit message: footprints asignados
Parts:
- U12: footprint Package_SO:SSOP-24_5.3x8.2mm_P0.65mm -> Package_SO:Texas_HTSOP-8-1EP_3.9x4.9mm_P1.27mm_EP2.95x4.9mm_Mask2.4x3.1mm_ThermalVias
Changed lines of the file:
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@@
 			)
 		)
-		(property "Footprint" "Package_SO:SSOP-24_5.3x8.2mm_P0.65mm"
+		(property "Footprint" "Package_SO:Texas_HTSOP-8-1EP_3.9x4.9mm_P1.27mm_EP2.95x4.9mm_Mask2.4x3.1mm_ThermalVias"
 			(at 199.39 59.69 0)
 			(effects
