File: KiCad/MÒDULMAX3232.kicad_sch (KiCad schematic)
At the start: 0 parts

Commit message: Arreglats errors i modificació del microcontrolador
Parts:
- added C18, C19, C21, C22: 100 nF, symbol Device:C
- added C7: C, symbol Device:C
- added U3: MAX3232, symbol Interface_UART:MAX3232
Connections:
- new net: C18.1, U3.1 (C1+)
- new net: C18.2, U3.3 (C1-)
- new net: C22.1, U3.6 (VS-)
- new net: C21.1, U3.2 (VS+)
- new net: C19.1, U3.4 (C2+)
- new net: C19.2, U3.5 (C2-)
- new net +3.3V: C21.2, C7.1, U3.16 (VCC)
- new net GND: C22.2, C7.2, U3.15 (GND)
- no-connect marks 0 -> 4

Commit message: Arreglat lo del MAX
Parts:
- C100: renamed from C7; value C -> 100 nF
- renumbered C18 to C101, C19 to C103, C21 to C104, C22 to C105, U3 to U20
Connections:
- net UART_TX: now reaches U20.11 (T1IN)
- net UART_RX: now reaches U20.12 (R1OUT)
- net RX: now reaches U20.13 (R1IN)
- net TX: now reaches U20.14 (T1OUT)

Commit message: Cambio en la parte de motores y drivers
Parts:
- renumbered C101 to C18, C103 to C19, C104 to C21, C105 to C22, C100 to C7, U20 to U3
Changed lines of the file:
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@@
 		(dnp no)
 		(fields_autoplaced yes)
-		(property "Reference" "#FLG03"
+		(property "Reference" "#FLG?"
 			(at 123.19 83.185 0)
 			(effects
@@
 				)
 			)
+			(project "SEIENTS_EDD"
+				(path "/b6401b4f-5426-49b8-bb2e-8ecdb19989ef/cbe76028-86be-49de-be25-b423cc5e8950"
+					(reference "#FLG?")
+					(unit 1)
+				)
+			)
 		)
 	)
@@
 		(on_board yes)
 		(dnp no)
-		(property "Reference" "C100"
+		(property "Reference" "C7"
 			(at 126.238 44.704 0)
 			(effects
@@
 		(on_board yes)
 		(dnp no)
-		(property "Reference" "#FLG04"
+		(property "Reference" "#FLG?"
 			(at 163.83 97.155 0)
 			(effects
@@
 				)
 			)
+			(project "SEIENTS_EDD"
+				(path "/b6401b4f-5426-49b8-bb2e-8ecdb19989ef/cbe76028-86be-49de-be25-b423cc5e8950"
+					(reference "#FLG?")
+					(unit 1)
+				)
+			)
 		)
 	)
@@
 		(on_board yes)
 		(dnp no)
-		(property "Reference" "#PWR0102"
+		(property "Reference" "#PWR030"
 			(at 134.62 57.15 0)
 			(effects
@@
 		(dnp no)
 		(fields_autoplaced yes)
-		(property "Reference" "#PWR0101"
+		(property "Reference" "#PWR011"
 			(at 143.51 124.46 0)
 			(effects
@@
 		(on_board yes)
 		(dnp no)
-		(property "Reference" "#FLG01"
+		(property "Reference" "#FLG?"
 			(at 145.415 46.99 0)
 			(effects
@@
 				)
 			)
+			(project "SEIENTS_EDD"
+				(path "/b6401b4f-5426-49b8-bb2e-8ecdb19989ef/cbe76028-86be-49de-be25-b423cc5e8950"
+					(reference "#FLG?")
+					(unit 1)
+				)
+			)
 		)
 	)
@@
 		(on_board yes)
 		(dnp no)
-		(property "Reference" "C101"
+		(property "Reference" "C18"
 			(at 115.316 62.738 0)
 			(effects
@@
 		(on_board yes)
 		(dnp no)
-		(property "Reference" "#PWR0103"
+		(property "Reference" "#PWR032"
 			(at 186.69 88.9 0)
 			(effects
@@
 		(on_board yes)
 		(dnp no)
-		(property "Reference" "C105"
+		(property "Reference" "C22"
 			(at 171.958 75.438 90)
 			(effects
@@
 		(on_board yes)
 		(dnp no)
-		(property "Reference" "C104"
+		(property "Reference" "C21"
 			(at 171.704 67.564 90)
 			(effects
@@
 		(dnp no)
 		(fields_autoplaced yes)
-		(property "Reference" "U20"
+		(property "Reference" "U3"
 			(at 145.6533 52.07 0)
 			(effects
@@
 		(dnp no)
 		(fields_autoplaced yes)
-		(property "Reference" "C103"
+		(property "Reference" "C19"
 			(at 167.64 62.2299 0)
 			(effects
@@
 		(dnp no)
 		(fields_autoplaced yes)
-		(property "Reference" "#FLG02"
+		(property "Reference" "#FLG?"
 			(at 145.415 118.11 0)
 			(effects
@@
 					(unit 1)
 				)
+			)
+			(project "SEIENTS_EDD"
+				(path "/b6401b4f-5426-49b8-bb2e-8ecdb19989ef/cbe76028-86be-49de-be25-b423cc5e8950"
+					(reference "#FLG?")
+					(unit 1)
+				)

Commit message: Modificacions Micro
Changed lines of the file:
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@@
 	(paper "A4")
-	(junction
-		(at 143.51 46.99)
-		(diameter 0)
-		(color 0 0 0 0)
-	)
 	(junction
 		(at 163.83 95.25)
@@
 	)
 	(junction
-		(at 123.19 85.09)
-		(diameter 0)
-		(color 0 0 0 0)
-	)
-	(junction
 		(at 143.51 118.11)
 		(diameter 0)
@@
 	(wire
 		(pts
-			(xy 143.51 39.37) (xy 143.51 46.99)
+			(xy 143.51 39.37) (xy 143.51 52.07)
 		)
 		(stroke
@@
 		(pts
 			(xy 143.51 113.03) (xy 143.51 118.11)
-		)
-		(stroke
-			(width 0)
-			(type default)
-		)
-	)
-	(wire
-		(pts
-			(xy 143.51 46.99) (xy 143.51 52.07)
 		)
 		(stroke
@@
 	)
 	(global_label "UART_RX"
-		(shape output)
+		(shape bidirectional)
 		(at 118.11 95.25 180)
 		(fields_autoplaced yes)
@@
 		)
 		(property "Intersheetrefs" "${INTERSHEET_REFS}"
-			(at 107.021 95.25 0)
+			(at 106.7227 95.25 0)
 			(effects
 				(font
@@
 				(justify right)
 				(hide yes)
-			)
-		)
-	)
-	(symbol
-		(lib_id "power:PWR_FLAG")
-		(at 123.19 85.09 0)
-		(unit 1)
-		(exclude_from_sim no)
-		(in_bom yes)
-		(on_board yes)
-		(dnp no)
-		(fields_autoplaced yes)
-		(property "Reference" "#FLG?"
-			(at 123.19 83.185 0)
-			(effects
-				(font
-					(size 1.27 1.27)
-				)
-				(hide yes)
-			)
-		)
-		(property "Value" "PWR_FLAG"
-			(at 123.19 80.01 0)
-			(effects
-				(font
-					(size 1.27 1.27)
-				)
-			)
-		)
-		(property "Footprint" ""
-			(at 123.19 85.09 0)
-			(effects
-				(font
-					(size 1.27 1.27)
-				)
-				(hide yes)
-			)
-		)
-		(property "Datasheet" "~"
-			(at 123.19 85.09 0)
-			(effects
-				(font
-					(size 1.27 1.27)
-				)
-				(hide yes)
-			)
-		)
-		(property "Description" "Special symbol for telling ERC where power comes from"
-			(at 123.19 85.09 0)
-			(effects
-				(font
-					(size 1.27 1.27)
-				)
-				(hide yes)
-			)
-		)
-		(pin "1"
-		)
-		(instances
-			(project "MÒDULMAX3232"
-				(path "/31976a33-0b7e-4d28-8e87-80fe20812731"
-					(reference "#FLG03")
-					(unit 1)
-				)
-			)
-			(project "SEIENTS_EDD"
-				(path "/b6401b4f-5426-49b8-bb2e-8ecdb19989ef/cbe76028-86be-49de-be25-b423cc5e8950"
-					(reference "#FLG?")
-					(unit 1)
-				)
 			)
 		)
@@
 		(on_board yes)
 		(dnp no)
-		(property "Reference" "#FLG?"
+		(property "Reference" "#FLG022"
 			(at 163.83 97.155 0)
 			(effects
@@
 			(project "SEIENTS_EDD"
 				(path "/b6401b4f-5426-49b8-bb2e-8ecdb19989ef/cbe76028-86be-49de-be25-b423cc5e8950"
-					(reference "#FLG?")
+					(reference "#FLG022")
 					(unit 1)
 				)
@@
 	)
 	(symbol
-		(lib_id "power:PWR_FLAG")
-		(at 143.51 46.99 270)
-		(unit 1)
-		(exclude_from_sim no)
-		(in_bom yes)
-		(on_board yes)
-		(dnp no)
-		(property "Reference" "#FLG?"
-			(at 145.415 46.99 0)
-			(effects
-				(font
-					(size 1.27 1.27)
-				)
-				(hide yes)
-			)
-		)
-		(property "Value" "PWR_FLAG"
-			(at 145.542 44.958 90)
-			(effects
-				(font
-					(size 1.27 1.27)
-				)
-				(justify left)
-			)
-		)
-		(property "Footprint" ""
-			(at 143.51 46.99 0)
-			(effects
-				(font
-					(size 1.27 1.27)
-				)
-				(hide yes)
-			)
-		)
-		(property "Datasheet" "~"
-			(at 143.51 46.99 0)
-			(effects
-				(font
-					(size 1.27 1.27)
-				)
-				(hide yes)
-			)
-		)
-		(property "Description" "Special symbol for telling ERC where power comes from"
-			(at 143.51 46.99 0)
-			(effects
-				(font
-					(size 1.27 1.27)
-				)
-				(hide yes)
-			)
-		)
-		(pin "1"
-		)
-		(instances
-			(project ""
-				(path "/31976a33-0b7e-4d28-8e87-80fe20812731"
-					(reference "#FLG01")
-					(unit 1)
-				)
-			)
-			(project "SEIENTS_EDD"
-				(path "/b6401b4f-5426-49b8-bb2e-8ecdb19989ef/cbe76028-86be-49de-be25-b423cc5e8950"
-					(reference "#FLG?")
-					(unit 1)
-				)
-			)
-		)
-	)
-	(symbol
 		(lib_id "Device:C")
 		(at 123.19 63.5 0)
@@
 		(dnp no)
 		(fields_autoplaced yes)
-		(property "Reference" "#FLG?"
+		(property "Reference" "#FLG021"
 			(at 145.415 118.11 0)
 			(effects
@@
 			(project "SEIENTS_EDD"
 				(path "/b6401b4f-5426-49b8-bb2e-8ecdb19989ef/cbe76028-86be-49de-be25-b423cc5e8950"
-					(reference "#FLG?")
-					(unit 1)
-				)
+					(reference "#FLG021")
+					(unit 1)
+				)

Commit message: Començat el LAYOUT
Parts:
- U3: footprint (none) -> Connector_PinHeader_2.54mm:PinHeader_1x04_P2.54mm_Vertical
Changed lines of the file:
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@@
 			)
 		)
-		(property "Footprint" ""
+		(property "Footprint" "Connector_PinHeader_2.54mm:PinHeader_1x04_P2.54mm_Vertical"
 			(at 144.78 109.22 0)
 			(effects

Commit message: footprints asignados
Parts:
- C18, C19, C21, C22, C7: footprint (none) -> Capacitor_SMD:C_0805_2012Metric
- U3: footprint Connector_PinHeader_2.54mm:PinHeader_1x04_P2.54mm_Vertical -> Package_SO:SOIC-16_3.9x9.9mm_P1.27mm
Changed lines of the file:
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@@
 			)
 		)
-		(property "Footprint" ""
+		(property "Footprint" "Capacitor_SMD:C_0805_2012Metric"
 			(at 135.5852 49.53 0)
 			(effects
@@
 			)
 		)
-		(property "Footprint" ""
+		(property "Footprint" "Capacitor_SMD:C_0805_2012Metric"
 			(at 124.1552 67.31 0)
 			(effects
@@
 			)
 		)
-		(property "Footprint" ""
+		(property "Footprint" "Capacitor_SMD:C_0805_2012Metric"
 			(at 171.45 79.0448 0)
 			(effects
@@
 			)
 		)
-		(property "Footprint" ""
+		(property "Footprint" "Capacitor_SMD:C_0805_2012Metric"
 			(at 171.45 71.4248 0)
 			(effects
@@
 			)
 		)
-		(property "Footprint" "Connector_PinHeader_2.54mm:PinHeader_1x04_P2.54mm_Vertical"
+		(property "Footprint" "Package_SO:SOIC-16_3.9x9.9mm_P1.27mm"
 			(at 144.78 109.22 0)
 			(effects
@@
 			)
 		)
-		(property "Footprint" ""
+		(property "Footprint" "Capacitor_SMD:C_0805_2012Metric"
 			(at 164.7952 67.31 0)
 			(effects

Commit message: Modificat ETIQUETES MICROCONTROLADOR i errors varis
Changed lines of the file:
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@@
-	)
-	(junction
-		(at 143.51 118.11)
-		(diameter 0)
-		(color 0 0 0 0)
 	)
 	(junction
@@
 					(unit 1)
 				)
-			)
-		)
-	)
-	(symbol
-		(lib_id "power:PWR_FLAG")
-		(at 143.51 118.11 270)
-		(unit 1)
-		(exclude_from_sim no)
-		(in_bom yes)
-		(on_board yes)
-		(dnp no)
-		(fields_autoplaced yes)
-		(property "Reference" "#FLG021"
-			(at 145.415 118.11 0)
-			(effects
-				(font
-					(size 1.27 1.27)
-				)
-				(hide yes)
-			)
-		)
-		(property "Value" "PWR_FLAG"
-			(at 147.32 118.1099 90)
-			(effects
-				(font
-					(size 1.27 1.27)
-				)
-				(justify left)
-			)
-		)
-		(property "Footprint" ""
-			(at 143.51 118.11 0)
-			(effects
-				(font
-					(size 1.27 1.27)
-				)
-				(hide yes)
-			)
-		)
-		(property "Datasheet" "~"
-			(at 143.51 118.11 0)
-			(effects
-				(font
-					(size 1.27 1.27)
-				)
-				(hide yes)
-			)
-		)
-		(property "Description" "Special symbol for telling ERC where power comes from"
-			(at 143.51 118.11 0)
-			(effects
-				(font
-					(size 1.27 1.27)
-				)
-				(hide yes)
-			)
-		)
-		(pin "1"
-		)
-		(instances
-			(project "MÒDULMAX3232"
-				(path "/31976a33-0b7e-4d28-8e87-80fe20812731"
-					(reference "#FLG02")
-					(unit 1)
-				)
-			)
-			(project "SEIENTS_EDD"
-				(path "/b6401b4f-5426-49b8-bb2e-8ecdb19989ef/cbe76028-86be-49de-be25-b423cc5e8950"
-					(reference "#FLG021")
-					(unit 1)
-				)
