File: KiCad/POTENCIA.kicad_sch (KiCad schematic)
At the start: 23 parts

Commit message: Modificació al placement
Parts:
- gave numbers to parts that had none: 15
- renumbered C1 to C304, R1 to R209, R2 to R210, R3 to R211
Changed lines of the file:
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@@
 		(dnp no)
 		(fields_autoplaced yes)
-		(property "Reference" "R?"
+		(property "Reference" "R24"
 			(at 93.98 140.9699 0)
 			(effects
@@
 		(dnp no)
 		(fields_autoplaced yes)
-		(property "Reference" "#PWR?"
+		(property "Reference" "#PWR048"
 			(at 64.77 104.14 0)
 			(effects
@@
 		(dnp no)
 		(fields_autoplaced yes)
-		(property "Reference" "R?"
+		(property "Reference" "R23"
 			(at 132.08 101.6 90)
 			(effects
@@
 		(on_board yes)
 		(dnp no)
-		(property "Reference" "Q?"
+		(property "Reference" "Q201"
 			(at 202.184 96.774 0)
 			(effects
@@
 		(dnp no)
 		(fields_autoplaced yes)
-		(property "Reference" "U?"
+		(property "Reference" "U5"
 			(at 71.9933 86.36 0)
 			(effects
@@
 		(dnp no)
 		(fields_autoplaced yes)
-		(property "Reference" "#PWR?"
+		(property "Reference" "#PWR055"
 			(at 146.05 118.11 0)
 			(effects
@@
 				)
 			)
+			(project "SEIENTS_EDD"
+				(path "/b6401b4f-5426-49b8-bb2e-8ecdb19989ef/59990b35-698c-4572-9d1a-e1ee1d49a527"
+					(reference "C301")
+					(unit 1)
+				)
+			)
 		)
 	)
@@
 		(dnp no)
 		(fields_autoplaced yes)
-		(property "Reference" "#PWR02"
+		(property "Reference" "#PWR0106"
 			(at 254 134.62 0)
 			(effects
@@
 		(dnp no)
 		(fields_autoplaced yes)
-		(property "Reference" "U?"
+		(property "Reference" "U7"
 			(at 49.1333 119.38 0)
 			(effects
@@
 		(dnp no)
 		(fields_autoplaced yes)
-		(property "Reference" "#PWR?"
+		(property "Reference" "#PWR053"
 			(at 91.44 157.48 0)
 			(effects
@@
 		(dnp no)
 		(fields_autoplaced yes)
-		(property "Reference" "M?"
+		(property "Reference" "M5"
 			(at 95.25 72.3899 0)
 			(effects
@@
 		(dnp no)
 		(fields_autoplaced yes)
-		(property "Reference" "#PWR?"
+		(property "Reference" "#PWR049"
 			(at 26.67 147.32 0)
 			(effects
@@
 		(dnp no)
 		(fields_autoplaced yes)
-		(property "Reference" "#FLG?"
+		(property "Reference" "#FLG05"
 			(at 95.25 19.685 0)
 			(effects
@@
 		(dnp no)
 		(fields_autoplaced yes)
-		(property "Reference" "C1"
+		(property "Reference" "C304"
 			(at 121.92 71.1199 0)
 			(effects
@@
 				)
 			)
+			(project "SEIENTS_EDD"
+				(path "/b6401b4f-5426-49b8-bb2e-8ecdb19989ef/59990b35-698c-4572-9d1a-e1ee1d49a527"
+					(reference "C304")
+					(unit 1)
+				)
+			)
 		)
 	)
@@
 		(on_board yes)
 		(dnp no)
-		(property "Reference" "M?"
+		(property "Reference" "M4"
 			(at 95.25 57.1499 0)
 			(effects
@@
 		(dnp no)
 		(fields_autoplaced yes)
-		(property "Reference" "#PWR01"
+		(property "Reference" "#PWR0102"
 			(at 213.36 134.62 0)
 			(effects
@@
 		(dnp no)
 		(fields_autoplaced yes)
-		(property "Reference" "D?"
+		(property "Reference" "D100"
 			(at 256.54 118.4274 90)
 			(effects
@@
 		(dnp no)
 		(fields_autoplaced yes)
-		(property "Reference" "R3"
+		(property "Reference" "R211"
 			(at 256.54 106.6799 0)
 			(effects
@@
 				)
 			)
+			(project "SEIENTS_EDD"
+				(path "/b6401b4f-5426-49b8-bb2e-8ecdb19989ef/59990b35-698c-4572-9d1a-e1ee1d49a527"
+					(reference "C300")
+					(unit 1)
+				)
+			)
 		)
 	)
@@
 		(dnp no)
 		(fields_autoplaced yes)
-		(property "Reference" "J?"
+		(property "Reference" "J201"
 			(at 217.17 73.66 90)
 			(effects
@@
 		(dnp no)
 		(fields_autoplaced yes)
-		(property "Reference" "R1"
+		(property "Reference" "R209"
 			(at 203.2 111.7599 0)
 			(effects
@@
 		(dnp no)
 		(fields_autoplaced yes)
-		(property "Reference" "U?"
+		(property "Reference" "U8"
 			(at 116.4433 83.82 0)
 			(effects
@@
 		(dnp no)
 		(fields_autoplaced yes)
-		(property "Reference" "C?"
+		(property "Reference" "C32"
 			(at 30.48 134.6199 0)
 			(effects
@@
 		(dnp no)
 		(fields_autoplaced yes)
-		(property "Reference" "#PWR?"
+		(property "Reference" "#PWR050"
 			(at 46.99 176.53 0)
 			(effects
@@
 		(dnp no)
 		(fields_autoplaced yes)
-		(property "Reference" "R?"
+		(property "Reference" "R14"
 			(at 80.01 119.3801 0)
 			(effects
@@
 		(dnp no)
 		(fields_autoplaced yes)
-		(property "Reference" "R?"
+		(property "Reference" "R1"
 			(at 67.31 120.6499 0)
 			(effects
@@
 		(dnp no)
 		(fields_autoplaced yes)
-		(property "Reference" "R?"
+		(property "Reference" "R26"
 			(at 96.52 120.6499 0)
 			(effects
@@
 		(dnp no)
 		(fields_autoplaced yes)
-		(property "Reference" "M?"
+		(property "Reference" "M6"
 			(at 142.24 92.7099 0)
 			(effects
@@
 		(dnp no)
 		(fields_autoplaced yes)
-		(property "Reference" "#PWR?"
+		(property "Reference" "#PWR051"
 			(at 114.3 118.11 0)
 			(effects
@@
 		(dnp no)
 		(fields_autoplaced yes)
-		(property "Reference" "R2"
+		(property "Reference" "R210"
 			(at 227.33 82.55 90)
 			(effects
@@
 				)
 			)
+			(project "SEIENTS_EDD"
+				(path "/b6401b4f-5426-49b8-bb2e-8ecdb19989ef/59990b35-698c-4572-9d1a-e1ee1d49a527"
+					(reference "C303")
+					(unit 1)
+				)
+			)
 		)
 	)
@@
 					(reference "C302")
 					(unit 1)
+				)
+			)
+			(project "SEIENTS_EDD"
+				(path "/b6401b4f-5426-49b8-bb2e-8ecdb19989ef/59990b35-698c-4572-9d1a-e1ee1d49a527"
+					(reference "C302")
+					(unit 1)

Commit message: Modificació al placement
Connections:
- net +3.3V: now also C32.2
- net GND: no longer C32.2
Other:
- moved on the sheet: C32
Changed lines of the file:
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@@
 	)
 	(junction
+		(at 46.99 116.84)
+		(diameter 0)
+		(color 0 0 0 0)
+	)
+	(junction
 		(at 43.18 29.21)
 		(diameter 0)
@@
 	)
 	(junction
+		(at 46.99 109.22)
+		(diameter 0)
+		(color 0 0 0 0)
+	)
+	(junction
 		(at 64.77 95.25)
 		(diameter 0)
@@
 	(wire
 		(pts
-			(xy 26.67 139.7) (xy 26.67 140.97)
+			(xy 46.99 109.22) (xy 46.99 116.84)
 		)
 		(stroke
@@
 	(wire
 		(pts
+			(xy 39.37 116.84) (xy 46.99 116.84)
+		)
+		(stroke
+			(width 0)
+			(type default)
+		)
+	)
+	(wire
+		(pts
 			(xy 54.61 95.25) (xy 64.77 95.25)
 		)
@@
 	(wire
 		(pts
+			(xy 46.99 116.84) (xy 46.99 121.92)
+		)
+		(stroke
+			(width 0)
+			(type default)
+		)
+	)
+	(wire
+		(pts
 			(xy 91.44 146.05) (xy 91.44 151.13)
 		)
@@
 	(wire
 		(pts
-			(xy 46.99 120.65) (xy 46.99 121.92)
+			(xy 46.99 104.14) (xy 46.99 109.22)
 		)
 		(stroke
@@
 	(wire
 		(pts
-			(xy 26.67 129.54) (xy 26.67 132.08)
-		)
-		(stroke
-			(width 0)
-			(type default)
-		)
-	)
-	(wire
-		(pts
 			(xy 90.17 66.04) (xy 77.47 66.04)
 		)
@@
 		)
 	)
+	(wire
+		(pts
+			(xy 39.37 109.22) (xy 46.99 109.22)
+		)
+		(stroke
+			(width 0)
+			(type default)
+		)
+	)
 	(polyline
 		(pts
@@
 	(global_label "+3.3V"
 		(shape input)
-		(at 46.99 120.65 90)
+		(at 46.99 104.14 90)
 		(fields_autoplaced yes)
 		(effects
@@
 		)
 		(property "Intersheetrefs" "${INTERSHEET_REFS}"
-			(at 46.99 111.98 90)
+			(at 46.99 95.47 90)
 			(effects
 				(font
@@
 	(global_label "+3.3V"
 		(shape input)
-		(at 26.67 129.54 180)
-		(fields_autoplaced yes)
-		(effects
-			(font
-				(size 1.27 1.27)
-			)
-			(justify right)
-		)
-		(property "Intersheetrefs" "${INTERSHEET_REFS}"
-			(at 18 129.54 0)
-			(effects
-				(font
-					(size 1.27 1.27)
-				)
-				(justify right)
-				(hide yes)
-			)
-		)
-	)
-	(global_label "+3.3V"
-		(shape input)
 		(at 64.77 115.57 90)
 		(fields_autoplaced yes)
@@
 	)
 	(symbol
-		(lib_id "power:GND")
-		(at 26.67 140.97 0)
-		(unit 1)
-		(exclude_from_sim no)
-		(in_bom yes)
-		(on_board yes)
-		(dnp no)
-		(fields_autoplaced yes)
-		(property "Reference" "#PWR049"
-			(at 26.67 147.32 0)
-			(effects
-				(font
-					(size 1.27 1.27)
-				)
-				(hide yes)
-			)
-		)
-		(property "Value" "GND"
-			(at 26.67 146.05 0)
-			(effects
-				(font
-					(size 1.27 1.27)
-				)
-			)
-		)
-		(property "Footprint" ""
-			(at 26.67 140.97 0)
-			(effects
-				(font
-					(size 1.27 1.27)
-				)
-				(hide yes)
-			)
-		)
-		(property "Datasheet" ""
-			(at 26.67 140.97 0)
-			(effects
-				(font
-					(size 1.27 1.27)
-				)
-				(hide yes)
-			)
-		)
-		(property "Description" "Power symbol creates a global label with name \"GND\" , ground"
-			(at 26.67 140.97 0)
-			(effects
-				(font
-					(size 1.27 1.27)
-				)
-				(hide yes)
-			)
-		)
-		(pin "1"
-		)
-		(instances
-			(project "POTENCIA"
-				(path "/6c7f9d9d-0dea-474c-bc2e-f5f0ea810945"
-					(reference "#PWR?")
-					(unit 1)
-				)
-			)
-			(project "SEIENTS_EDD"
-				(path "/b6401b4f-5426-49b8-bb2e-8ecdb19989ef/59990b35-698c-4572-9d1a-e1ee1d49a527"
-					(reference "#PWR049")
-					(unit 1)
-				)
-			)
-		)
-	)
-	(symbol
 		(lib_id "power:PWR_FLAG")
 		(at 95.25 17.78 180)
@@
 	(symbol
 		(lib_id "Device:C")
-		(at 26.67 135.89 0)
+		(at 39.37 113.03 0)
 		(unit 1)
 		(exclude_from_sim no)
@@
 		(on_board yes)
 		(dnp no)
-		(fields_autoplaced yes)
 		(property "Reference" "C32"
-			(at 30.48 134.6199 0)
+			(at 29.718 111.76 0)
 			(effects
 				(font
@@
 		)
 		(property "Value" "100nF"
-			(at 30.48 137.1599 0)
+			(at 29.718 114.3 0)
 			(effects
 				(font
@@
 		)
 		(property "Footprint" "Capacitor_SMD:C_0805_2012Metric"
-			(at 27.6352 139.7 0)
+			(at 40.3352 116.84 0)
 			(effects
 				(font
@@
 		)
 		(property "Datasheet" "~"
-			(at 26.67 135.89 0)
+			(at 39.37 113.03 0)
 			(effects
 				(font
@@
 		)
 		(property "Description" "Unpolarized capacitor"
-			(at 26.67 135.89 0)
+			(at 39.37 113.03 0)
 			(effects
 				(font

Commit message: Routing V1
Connections:
- net POS_IN1: now also U5.22 (AIN2); no longer U5.21 (AIN1)
- net POS_IN2: now also U5.21 (AIN1); no longer U5.22 (AIN2)
- net VBAT: no longer J201.2 (Pin_2)
- no-connect marks 6 -> 7
Changed lines of the file:
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@@
+	)
+	(no_connect
+		(at 215.9 85.09)
 	)
 	(no_connect
@@
 	(global_label "POS_IN1"
 		(shape input)
-		(at 34.29 66.04 180)
+		(at 34.29 68.58 180)
 		(fields_autoplaced yes)
 		(effects
@@
 		)
 		(property "Intersheetrefs" "${INTERSHEET_REFS}"
-			(at 24.0366 66.04 0)
+			(at 24.0366 68.58 0)
 			(effects
 				(font
@@
 				)
 				(justify left)
-				(hide yes)
-			)
-		)
-	)
-	(global_label "VBAT"
-		(shape input)
-		(at 215.9 85.09 270)
-		(fields_autoplaced yes)
-		(effects
-			(font
-				(size 1.27 1.27)
-			)
-			(justify right)
-		)
-		(property "Intersheetrefs" "${INTERSHEET_REFS}"
-			(at 215.9 91.8358 90)
-			(effects
-				(font
-					(size 1.27 1.27)
-				)
-				(justify right)
 				(hide yes)
 			)
@@
 	(global_label "POS_IN2"
 		(shape input)
-		(at 34.29 68.58 180)
+		(at 34.29 66.04 180)
 		(fields_autoplaced yes)
 		(effects
@@
 		)
 		(property "Intersheetrefs" "${INTERSHEET_REFS}"
-			(at 23.3824 68.58 0)
-			(effects
-				(font
+			(at 23.3824 66.04 0)
+			(effects
+				(font
