File: KiCad/POTENCIA.kicad_sch (KiCad schematic)
At the start: 23 parts, among them J201 Screw_Terminal_01x04, M4 Motor_DC, M5 Motor_DC, M6 Motor_DC, Q201 IRLZ44N, U5 TB6612FNG, U7 ATtiny1616-M, U8 DRV8871DDA

Commit message: Modificació al routing
Connections:
- net +3.3V: no longer C300.2, C301.2, C32.2
- net GND: now also C302.2, C303.2, C304.2, C32.2
- net VBAT: no longer C302.1, C302.2, C303.1, C303.2, C304.2, U5.13 (VM2), U5.14 (VM3), U5.24 (VM1)
- net at U5.11 (BO1), U5.12 (BO1): now also M5.2 (-); no longer M5.1 (+)
- net at U5.7 (BO2), U5.8 (BO2): now also M5.1 (+); no longer M5.2 (-)
- new net: C300.2, C301.2
- new net VBAT/FUSE: C302.1, C303.1, U5.13 (VM2), U5.14 (VM3), U5.24 (VM1)
Other:
- moved on the sheet: M5

Commit message: Modificació al routing
Parts:
- renumbered C304 to C1, C32 to C?, D100 to D?, J201 to J?, M5 to M?, M4 to M?, M6 to M?, Q201 to Q?, R209 to R1, R210 to R2, R211 to R3, R24 to R?, R23 to R?, R14 to R?, R1 to R?, R26 to R?, U5 to U?, U7 to U?, U8 to U?
Connections:
- net GND: now also C300.2, C301.2
Changed lines of the file:
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@@
 	)
 	(junction
+		(at 39.37 36.83)
+		(diameter 0)
+		(color 0 0 0 0)
+	)
+	(junction
 		(at 82.55 132.08)
 		(diameter 0)
@@
 	(wire
 		(pts
+			(xy 39.37 36.83) (xy 39.37 38.1)
+		)
+		(stroke
+			(width 0)
+			(type default)
+		)
+	)
+	(wire
+		(pts
 			(xy 34.29 58.42) (xy 46.99 58.42)
 		)
@@
 	(wire
 		(pts
-			(xy 35.56 36.83) (xy 43.18 36.83)
+			(xy 35.56 36.83) (xy 39.37 36.83)
 		)
 		(stroke
@@
 	(wire
 		(pts
+			(xy 39.37 36.83) (xy 43.18 36.83)
+		)
+		(stroke
+			(width 0)
+			(type default)
+		)
+	)
+	(wire
+		(pts
 			(xy 78.74 26.67) (xy 85.09 26.67)
 		)
@@
 		(dnp no)
 		(fields_autoplaced yes)
-		(property "Reference" "#PWR020"
+		(property "Reference" "#PWR?"
 			(at 78.74 35.56 0)
 			(effects
@@
 		)
 		(instances
+			(project "POTENCIA"
+				(path "/6c7f9d9d-0dea-474c-bc2e-f5f0ea810945"
+					(reference "#PWR?")
+					(unit 1)
+				)
+			)
 			(project "SEIENTS_EDD"
 				(path "/b6401b4f-5426-49b8-bb2e-8ecdb19989ef/59990b35-698c-4572-9d1a-e1ee1d49a527"
@@
 		(dnp no)
 		(fields_autoplaced yes)
-		(property "Reference" "#PWR011"
+		(property "Reference" "#PWR?"
 			(at 39.37 123.19 0)
 			(effects
@@
 		)
 		(instances
+			(project "POTENCIA"
+				(path "/6c7f9d9d-0dea-474c-bc2e-f5f0ea810945"
+					(reference "#PWR?")
+					(unit 1)
+				)
+			)
 			(project ""
 				(path "/b6401b4f-5426-49b8-bb2e-8ecdb19989ef/59990b35-698c-4572-9d1a-e1ee1d49a527"
@@
 		(dnp no)
 		(fields_autoplaced yes)
-		(property "Reference" "R24"
+		(property "Reference" "R?"
 			(at 93.98 140.9699 0)
 			(effects
@@
 		(dnp no)
 		(fields_autoplaced yes)
-		(property "Reference" "#PWR048"
+		(property "Reference" "#PWR?"
 			(at 64.77 104.14 0)
 			(effects
@@
 		(dnp no)
 		(fields_autoplaced yes)
-		(property "Reference" "R23"
+		(property "Reference" "R?"
 			(at 132.08 101.6 90)
 			(effects
@@
 		(on_board yes)
 		(dnp no)
-		(property "Reference" "Q201"
+		(property "Reference" "Q?"
 			(at 202.184 96.774 0)
 			(effects
@@
 		(dnp no)
 		(fields_autoplaced yes)
-		(property "Reference" "U5"
+		(property "Reference" "U?"
 			(at 71.9933 86.36 0)
 			(effects
@@
 		(dnp no)
 		(fields_autoplaced yes)
-		(property "Reference" "#PWR055"
+		(property "Reference" "#PWR?"
 			(at 146.05 118.11 0)
 			(effects
@@
 		(dnp no)
 		(fields_autoplaced yes)
-		(property "Reference" "#PWR0106"
+		(property "Reference" "#PWR02"
 			(at 254 134.62 0)
 			(effects
@@
 		(dnp no)
 		(fields_autoplaced yes)
-		(property "Reference" "U7"
+		(property "Reference" "U?"
 			(at 49.1333 119.38 0)
 			(effects
@@
 		(dnp no)
 		(fields_autoplaced yes)
-		(property "Reference" "#PWR053"
+		(property "Reference" "#PWR?"
 			(at 91.44 157.48 0)
 			(effects
@@
 		(dnp no)
 		(fields_autoplaced yes)
-		(property "Reference" "M5"
+		(property "Reference" "M?"
 			(at 95.25 69.8499 0)
 			(effects
@@
 		(dnp no)
 		(fields_autoplaced yes)
-		(property "Reference" "#FLG05"
+		(property "Reference" "#FLG?"
 			(at 95.25 19.685 0)
 			(effects
@@
 		(dnp no)
 		(fields_autoplaced yes)
-		(property "Reference" "C304"
+		(property "Reference" "C1"
 			(at 121.92 71.1199 0)
 			(effects
@@
 		(on_board yes)
 		(dnp no)
-		(property "Reference" "M4"
+		(property "Reference" "M?"
 			(at 95.25 57.1499 0)
 			(effects
@@
 		(dnp no)
 		(fields_autoplaced yes)
-		(property "Reference" "#PWR0102"
+		(property "Reference" "#PWR01"
 			(at 213.36 134.62 0)
 			(effects
@@
 		(dnp no)
 		(fields_autoplaced yes)
-		(property "Reference" "D100"
+		(property "Reference" "D?"
 			(at 256.54 118.4274 90)
 			(effects
@@
 		(dnp no)
 		(fields_autoplaced yes)
-		(property "Reference" "R211"
+		(property "Reference" "R3"
 			(at 256.54 106.6799 0)
 			(effects
@@
 		(dnp no)
 		(fields_autoplaced yes)
-		(property "Reference" "J201"
+		(property "Reference" "J?"
 			(at 217.17 73.66 90)
 			(effects
@@
 		(dnp no)
 		(fields_autoplaced yes)
-		(property "Reference" "R209"
+		(property "Reference" "R1"
 			(at 203.2 111.7599 0)
 			(effects
@@
 		(dnp no)
 		(fields_autoplaced yes)
-		(property "Reference" "U8"
+		(property "Reference" "U?"
 			(at 116.4433 83.82 0)
 			(effects
@@
 		(on_board yes)
 		(dnp no)
-		(property "Reference" "C32"
+		(property "Reference" "C?"
 			(at 29.718 111.76 0)
 			(effects
@@
 		(dnp no)
 		(fields_autoplaced yes)
-		(property "Reference" "#PWR050"
+		(property "Reference" "#PWR?"
 			(at 46.99 176.53 0)
 			(effects
@@
 		(dnp no)
 		(fields_autoplaced yes)
-		(property "Reference" "#PWR017"
+		(property "Reference" "#PWR?"
 			(at 118.11 82.55 0)
 			(effects
@@
 		)
 		(instances
+			(project "POTENCIA"
+				(path "/6c7f9d9d-0dea-474c-bc2e-f5f0ea810945"
+					(reference "#PWR?")
+					(unit 1)
+				)
+			)
 			(project "SEIENTS_EDD"
 				(path "/b6401b4f-5426-49b8-bb2e-8ecdb19989ef/59990b35-698c-4572-9d1a-e1ee1d49a527"
@@
 		(dnp no)
 		(fields_autoplaced yes)
-		(property "Reference" "R14"
+		(property "Reference" "R?"
 			(at 80.01 119.3801 0)
 			(effects
@@
 		(dnp no)
 		(fields_autoplaced yes)
-		(property "Reference" "R1"
+		(property "Reference" "R?"
 			(at 67.31 120.6499 0)
 			(effects
@@
 		(dnp no)
 		(fields_autoplaced yes)
-		(property "Reference" "R26"
+		(property "Reference" "R?"
 			(at 96.52 120.6499 0)
 			(effects
@@
 		(dnp no)
 		(fields_autoplaced yes)
-		(property "Reference" "M6"
+		(property "Reference" "M?"
 			(at 142.24 92.7099 0)
 			(effects
@@
 	(symbol
 		(lib_id "power:GND")
+		(at 39.37 38.1 0)
+		(unit 1)
+		(exclude_from_sim no)
+		(in_bom yes)
+		(on_board yes)
+		(dnp no)
+		(fields_autoplaced yes)
+		(property "Reference" "#PWR03"
+			(at 39.37 44.45 0)
+			(effects
+				(font
+					(size 1.27 1.27)
+				)
+				(hide yes)
+			)
+		)
+		(property "Value" "GND"
+			(at 39.37 43.18 0)
+			(effects
+				(font
+					(size 1.27 1.27)
+				)
+			)
+		)
+		(property "Footprint" ""
+			(at 39.37 38.1 0)
+			(effects
+				(font
+					(size 1.27 1.27)
+				)
+				(hide yes)
+			)
+		)
+		(property "Datasheet" ""
+			(at 39.37 38.1 0)
+			(effects
+				(font
+					(size 1.27 1.27)
+				)
+				(hide yes)
+			)
+		)
+		(property "Description" "Power symbol creates a global label with name \"GND\" , ground"
+			(at 39.37 38.1 0)
+			(effects
+				(font
+					(size 1.27 1.27)
+				)
+				(hide yes)
+			)
+		)
+		(pin "1"
+		)
+		(instances
+			(project ""
+				(path "/6c7f9d9d-0dea-474c-bc2e-f5f0ea810945"
+					(reference "#PWR03")
+					(unit 1)
+				)
+			)
+		)
+	)
+	(symbol
+		(lib_id "power:GND")
 		(at 114.3 111.76 0)
 		(unit 1)
@@
 		(dnp no)
 		(fields_autoplaced yes)
-		(property "Reference" "#PWR051"
+		(property "Reference" "#PWR?"
 			(at 114.3 118.11 0)
 			(effects
@@
 		(dnp no)
 		(fields_autoplaced yes)
-		(property "Reference" "R210"
+		(property "Reference" "R2"
 			(at 227.33 82.55 90)
 			(effects

Commit message: ROUTING FINAL
Parts:
- gave numbers to parts that had none: 15
- renumbered C1 to C304, R1 to R209, R2 to R210, R3 to R211
Connections:
- net ALT_IN1: now also U7.15 (PC0); no longer U7.16 (PC1)
- net ALT_IN2: now also U7.16 (PC1); no longer U7.15 (PC0)
- net POS_IN1: now also U7.13 (PB1); no longer U7.6 (PA5)
- net POS_IN2: now also U7.12 (PB2); no longer U7.7 (PA6)
- net POS_PWM: now also U7.14 (PB0); no longer U7.5 (PA4)
- net REC_IN1: now also U7.11 (PB3); no longer U7.13 (PB1)
- net REC_IN2: now also U7.10 (PB4); no longer U7.14 (PB0)
- net REC_PWM: now also U7.9 (PB5); no longer U7.8 (PA7)
Other:
- moved on the sheet: R1, R26
